Commit message: Point mesh references at the package, not one developer home directory
test_robot_body.urdf.xacro referenced all ten of its meshes through absolute
paths under /home/nitin-5090/Documents/DevEnv/jazzy_ws/IGVC_robot_2026/. That
path exists on exactly one machine, which has left the team. Everywhere else the
robot body loaded with no visual and no collision geometry, so the chassis,
wheels and caster were invisible to both RViz and any physics engine.

The meshes were in the repository the whole time, and the sibling part files
gps_antenna.urdf.xacro and rplidar_c1.urdf.xacro already used package:// URIs.
Only the body was never cleaned up after CAD export.

All five referenced .obj files and all six .mtl sidecars are present, and no .mtl
carries an absolute texture path. CMakeLists.txt already installs meshes and urdf
into share, so package:// resolves after a colcon build.

Verified by expanding the xacro and converting it with gz sdf: all eight mesh
URIs resolve, and the model produces ten collision and fourteen visual elements.
Note that gz sdf alone does not catch this, because sdformat does not check that
a mesh file exists until load time.

The same substitution is applied to the two generated flat URDFs.

Co-Authored-By: Claude Opus 5 <noreply@anthropic.com>

File: src/igvc_test_description/igvc_robot.urdf (robot description, URDF)
Before this commit: robot igvc_test_robot, 27 links, 26 joints
Links:
- link caster_raceway_link: geometry collision mesh filename=package://igvc_test_description/meshes/caster_raceway_link_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 scale=1. 1. 1.; visual mesh filename=package://igvc_test_description/meshes/caster_raceway_link_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 scale=1. 1. 1.
- link caster_wheel_link: geometry collision mesh filename=package://igvc_test_description/meshes/caster_wheel_link__i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 scale=1. 1. 1.; visual mesh filename=package://igvc_test_description/meshes/caster_wheel_link__i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 scale=1. 1. 1.
- link chassis_link: geometry collision mesh filename=package://igvc_test_description/meshes/_FE2CBA3_2B86_49A6_8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 scale=1. 1. 1.; visual mesh filename=package://igvc_test_description/meshes/_FE2CBA3_2B86_49A6_8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 scale=1. 1. 1.
- link front_zed_camera_x_camera_center: geometry collision mesh filename=package://igvc_test_description/meshes/zedx.stl; visual mesh filename=package://igvc_test_description/meshes/zedx.stl
- link left_wheel_link: geometry collision mesh filename=package://igvc_test_description/meshes/left_wheel_link__in_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 scale=1. 1. 1.; visual mesh filename=package://igvc_test_description/meshes/left_wheel_link__in_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 scale=1. 1. 1.
- link left_zed_camera_x_camera_center: geometry collision mesh filename=package://igvc_test_description/meshes/zedx.stl; visual mesh filename=package://igvc_test_description/meshes/zedx.stl
- link right_wheel_link: geometry collision mesh filename=package://igvc_test_description/meshes/right_wheel_link__in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 scale=1. 1. 1.; visual mesh filename=package://igvc_test_description/meshes/right_wheel_link__in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 scale=1. 1. 1.
- link right_zed_camera_x_camera_center: geometry collision mesh filename=package://igvc_test_description/meshes/zedx.stl; visual mesh filename=package://igvc_test_description/meshes/zedx.stl

File: src/igvc_test_description/test_robot.urdf (robot description, URDF)
Before this commit: robot igvc_test_robot, 29 links, 28 joints
Links:
- link caster_raceway_link: geometry collision mesh filename=package://igvc_test_description/meshes/caster_raceway_link_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 scale=1. 1. 1.; visual mesh filename=package://igvc_test_description/meshes/caster_raceway_link_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 scale=1. 1. 1.
- link caster_wheel_link: geometry collision mesh filename=package://igvc_test_description/meshes/caster_wheel_link__i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 scale=1. 1. 1.; visual mesh filename=package://igvc_test_description/meshes/caster_wheel_link__i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 scale=1. 1. 1.
- link chassis_link: geometry collision mesh filename=package://igvc_test_description/meshes/_FE2CBA3_2B86_49A6_8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 scale=1. 1. 1.; visual box size=0.05 0.05 0.3
- link front_zed_camera_x_camera_center: geometry collision mesh filename=package://igvc_test_description/meshes/zedx.stl; visual mesh filename=package://igvc_test_description/meshes/zedx.stl
- link left_wheel_link: geometry collision mesh filename=package://igvc_test_description/meshes/left_wheel_link__in_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 scale=1. 1. 1.; visual mesh filename=package://igvc_test_description/meshes/left_wheel_link__in_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 scale=1. 1. 1.
- link left_zed_camera_x_camera_center: geometry collision mesh filename=package://igvc_test_description/meshes/zedx.stl; visual mesh filename=package://igvc_test_description/meshes/zedx.stl
- link right_wheel_link: geometry collision mesh filename=package://igvc_test_description/meshes/right_wheel_link__in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 scale=1. 1. 1.; visual mesh filename=package://igvc_test_description/meshes/right_wheel_link__in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 scale=1. 1. 1.
- link right_zed_camera_x_camera_center: geometry collision mesh filename=package://igvc_test_description/meshes/zedx.stl; visual mesh filename=package://igvc_test_description/meshes/zedx.stl

File: src/igvc_test_description/urdf/parts/test_robot_body.urdf.xacro (robot description, xacro)
@@ -41,5 +41,5 @@
         <origin xyz="-0.0003886 -0.0011449 -0.0088217" rpy="0. 0. ${0.9071883-3.14152/4}" />
         <geometry>
-          <mesh filename="file:///home/nitin-5090/Documents/DevEnv/jazzy_ws/IGVC_robot_2026/src/igvc_test_description/meshes/caster_raceway_link_Part_2_Part_2.obj" scale="1. 1. 1." />
+          <mesh filename="package://igvc_test_description/meshes/caster_raceway_link_Part_2_Part_2.obj" scale="1. 1. 1." />
         </geometry>
       </visual>
@@ -47,5 +47,5 @@
         <origin xyz="-0.0003886 -0.0011449 -0.0088217" rpy="0. 0. ${0.9071883-3.14152/4}" />
         <geometry>
-          <mesh filename="file:///home/nitin-5090/Documents/DevEnv/jazzy_ws/IGVC_robot_2026/src/igvc_test_description/meshes/caster_raceway_link_Part_2_Part_2.obj" scale="1. 1. 1." />
+          <mesh filename="package://igvc_test_description/meshes/caster_raceway_link_Part_2_Part_2.obj" scale="1. 1. 1." />
         </geometry>
       </collision>
@@ -60,5 +60,5 @@
         <origin xyz="-0.1135063 0.0373062 -0.0238125" rpy="-1.570796 -1e-07 1.570796" />
         <geometry>
-          <mesh filename="file:///home/nitin-5090/Documents/DevEnv/jazzy_ws/IGVC_robot_2026/src/igvc_test_description/meshes/caster_wheel_link__in_Caster__in_Caster.obj" scale="1. 1. 1." />
+          <mesh filename="package://igvc_test_description/meshes/caster_wheel_link__in_Caster__in_Caster.obj" scale="1. 1. 1." />
         </geometry>
       </visual>
@@ -66,5 +66,5 @@
         <origin xyz="-0.1135063 0.0373062 -0.0238125" rpy="-1.570796 -1e-07 1.570796" />
         <geometry>
-          <mesh filename="file:///home/nitin-5090/Documents/DevEnv/jazzy_ws/IGVC_robot_2026/src/igvc_test_description/meshes/caster_wheel_link__in_Caster__in_Caster.obj" scale="1. 1. 1." />
+          <mesh filename="package://igvc_test_description/meshes/caster_wheel_link__in_Caster__in_Caster.obj" scale="1. 1. 1." />
         </geometry>
       </collision>
@@ -79,5 +79,5 @@
         <origin xyz="9.06e-05 -0.0010859 -0.0010079" rpy="0. 0.8801533 -3.141593" />
         <geometry>
-          <mesh filename="file:///home/nitin-5090/Documents/DevEnv/jazzy_ws/IGVC_robot_2026/src/igvc_test_description/meshes/left_wheel_link__in_Wheel_Stand_In_01__in_Wheel_Stand_In.obj" scale="1. 1. 1." />
+          <mesh filename="package://igvc_test_description/meshes/left_wheel_link__in_Wheel_Stand_In_01__in_Wheel_Stand_In.obj" scale="1. 1. 1." />
         </geometry>
       </visual>
@@ -85,5 +85,5 @@
         <origin xyz="9.06e-05 -0.0010859 -0.0010079" rpy="0. 0.8801533 -3.141593" />
         <geometry>
-          <mesh filename="file:///home/nitin-5090/Documents/DevEnv/jazzy_ws/IGVC_robot_2026/src/igvc_test_description/meshes/left_wheel_link__in_Wheel_Stand_In_01__in_Wheel_Stand_In.obj" scale="1. 1. 1." />
+          <mesh filename="package://igvc_test_description/meshes/left_wheel_link__in_Wheel_Stand_In_01__in_Wheel_Stand_In.obj" scale="1. 1. 1." />
         </geometry>
       </collision>
@@ -98,5 +98,5 @@
         <origin xyz="-0.0007409 0.0085441 0.0012195" rpy="-3.141593 0. -7.32051e-08" />
         <geometry>
-          <mesh filename="file:///home/nitin-5090/Documents/DevEnv/jazzy_ws/IGVC_robot_2026/src/igvc_test_description/meshes/right_wheel_link__in_Wheel_Stand_In_01__in_Wheel_Stand_In.obj" scale="1. 1. 1." />
+          <mesh filename="package://igvc_test_description/meshes/right_wheel_link__in_Wheel_Stand_In_01__in_Wheel_Stand_In.obj" scale="1. 1. 1." />
         </geometry>
       </visual>
@@ -104,5 +104,5 @@
         <origin xyz="-0.0007409 0.0085441 0.0012195" rpy="-3.141593 0. -7.32051e-08" />
         <geometry>
-          <mesh filename="file:///home/nitin-5090/Documents/DevEnv/jazzy_ws/IGVC_robot_2026/src/igvc_test_description/meshes/right_wheel_link__in_Wheel_Stand_In_01__in_Wheel_Stand_In.obj" scale="1. 1. 1." />
+          <mesh filename="package://igvc_test_description/meshes/right_wheel_link__in_Wheel_Stand_In_01__in_Wheel_Stand_In.obj" scale="1. 1. 1." />
         </geometry>
       </collision>
@@ -117,5 +117,5 @@
         <origin xyz="0. 0. 0." rpy="0. 0. 1.570796" />
         <geometry>
-          <mesh filename="file:///home/nitin-5090/Documents/DevEnv/jazzy_ws/IGVC_robot_2026/src/igvc_test_description/meshes/_FE2CBA3_2B86_49A6_86C6_46C335366A6A.obj" scale="1. 1. 1." />
+          <mesh filename="package://igvc_test_description/meshes/_FE2CBA3_2B86_49A6_86C6_46C335366A6A.obj" scale="1. 1. 1." />
         </geometry>
       </visual>
@@ -141,5 +141,5 @@
         <origin xyz="0. 0. 0." rpy="0. 0. 1.570796" />
         <geometry>
-          <mesh filename="file:///home/nitin-5090/Documents/DevEnv/jazzy_ws/IGVC_robot_2026/src/igvc_test_description/meshes/_FE2CBA3_2B86_49A6_86C6_46C335366A6A.obj" scale="1. 1. 1." />
+          <mesh filename="package://igvc_test_description/meshes/_FE2CBA3_2B86_49A6_86C6_46C335366A6A.obj" scale="1. 1. 1." />
         </geometry>
       </collision>
