Commit message: Four collision meshes have no vertex normals and segfault the physics engine
left_wheel, right_wheel, caster_wheel and caster_raceway have 528, 528, 500 and
209 vertices and ZERO vertex normals. Counted directly in the .obj files:

    caster_raceway_link_Part_2_Part_2.obj        209 verts,      0 normals
    caster_wheel_link__in_Caster__in_Caster.obj  500 verts,      0 normals
    left_wheel_link__in_Wheel_Stand_In...obj     528 verts,      0 normals
    right_wheel_link__in_Wheel_Stand_In..obj     528 verts,      0 normals
    _FE2CBA3_2B86_49A6_86C6_46C335366A6A.obj   73324 verts,  73324 normals

Loaded as collision geometry, dartsim reports "does not have a normal count [0]
that matches its vertex count [3168]. This submesh will be ignored!" and then
segfaults inside OdeMesh::fillArrays on the empty result. gz sim dies on the
first physics step with exit 139. Note 528 x 6 = 3168 and 500 x 6 = 3000,
exactly the counts in the error, which is how the four were identified.

Those four are precisely the parts that have to collide for the robot to move:
both drive wheels, the caster wheel and the bracket it swivels in. The chassis
mesh is fine. So the simulated robot could spawn and publish topics while being
unable to exist for one physics step.

The fix is simulation-only and the real robot's description is untouched. Under
sim:=true the four links get primitive colliders; under sim:=false they keep
their meshes exactly as before. Verified by expanding the xacro both ways:

    link                   sim:=true                    sim:=false
    left_wheel_link        cylinder r0.1016 l0.0640     mesh
    right_wheel_link       cylinder r0.1016 l0.0640     mesh
    caster_wheel_link      sphere r0.0801               mesh
    caster_raceway_link    none                         mesh

Primitives are the better answer even setting the crash aside. A faceted mesh
wheel rolls on its flats and catches on its edges, where a cylinder does not,
and RQ-11 notes that Gazebo mesh collision is expensive and costs real-time
factor directly. The raceway is a bracket that never touches the ground, so it
gets no collider rather than a guessed shape.

The numbers are measured, not invented. 0.1016 and 0.0640 are the wheel mesh's
own bounding box, which is also the evidence that controllers.yaml's
wheel_radius 0.2032 is the DIAMETER; see the existing note in
urdf/gazebo/gazebo_sim.urdf.xacro. 0.0801 is the caster radius implied by the
joint chain: the caster contacts the ground at -0.0307033 + -0.1223279 - 0.0801
= -0.2331, which is 4 mm below the drive wheels at -0.2290, and 4 mm is build
tolerance.

test_robot.urdf.xacro needed one unrelated change to make this possible. The
sim argument was declared at the bottom of the file, after <xacro:robot_body/>
had already run, so the body could not read it. Moved to the top, before every
include. Nothing else about the file changed.

The meshes themselves are still broken and this commit does not repair them.
Isaac Sim and any MoveIt planning load the same files. Whether to regenerate
them with normals, or to treat primitive colliders as the permanent answer for
simulation, is left open and recorded as outstanding item 16 in
docs/DOCKER_CHANGES.md.

Co-Authored-By: Claude Opus 5 <noreply@anthropic.com>

File: src/igvc_test_description/urdf/parts/test_robot_body.urdf.xacro (robot description, xacro)
@@ -44,10 +44,17 @@
         </geometry>
       </visual>
-      <collision>
-        <origin xyz="-0.0003886 -0.0011449 -0.0088217" rpy="0. 0. ${0.9071883-3.14152/4}" />
-        <geometry>
-          <mesh filename="package://igvc_test_description/meshes/caster_raceway_link_Part_2_Part_2.obj" scale="1. 1. 1." />
-        </geometry>
-      </collision>
+      <!-- SIM: no collider. This is the swivel bracket above the caster wheel;
+           it never touches the ground, and its mesh is one of the four with
+           zero vertex normals that crash dartsim (see the note on
+           left_wheel_link). Omitting it avoids both a bad guess at its shape
+           and a spurious contact. -->
+      <xacro:unless value="$(arg sim)">
+        <collision>
+          <origin xyz="-0.0003886 -0.0011449 -0.0088217" rpy="0. 0. ${0.9071883-3.14152/4}" />
+          <geometry>
+            <mesh filename="package://igvc_test_description/meshes/caster_raceway_link_Part_2_Part_2.obj" scale="1. 1. 1." />
+          </geometry>
+        </collision>
+      </xacro:unless>
     </link>
     <link name="caster_wheel_link">
@@ -63,10 +70,26 @@
         </geometry>
       </visual>
-      <collision>
-        <origin xyz="-0.1135063 0.0373062 -0.0238125" rpy="-1.570796 -1e-07 1.570796" />
-        <geometry>
-          <mesh filename="package://igvc_test_description/meshes/caster_wheel_link__in_Caster__in_Caster.obj" scale="1. 1. 1." />
-        </geometry>
-      </collision>
+      <!-- SIM: sphere. A sphere is the right collider for a caster anyway,
+           since it rolls in every direction without the mesh's facet edges
+           catching. Radius 0.0801 comes from the joint chain worked out in
+           urdf/gazebo/gazebo_sim.urdf.xacro: the caster contacts the ground at
+           -0.0307033 + -0.1223279 - 0.0801 = -0.2331, which is 4 mm below the
+           drive wheels at -0.2290. That 4 mm is build tolerance. -->
+      <xacro:if value="$(arg sim)">
+        <collision>
+          <origin xyz="0. 0. 0." rpy="0. 0. 0." />
+          <geometry>
+            <sphere radius="0.0801" />
+          </geometry>
+        </collision>
+      </xacro:if>
+      <xacro:unless value="$(arg sim)">
+        <collision>
+          <origin xyz="-0.1135063 0.0373062 -0.0238125" rpy="-1.570796 -1e-07 1.570796" />
+          <geometry>
+            <mesh filename="package://igvc_test_description/meshes/caster_wheel_link__in_Caster__in_Caster.obj" scale="1. 1. 1." />
+          </geometry>
+        </collision>
+      </xacro:unless>
     </link>
     <link name="left_wheel_link">
@@ -82,10 +105,36 @@
         </geometry>
       </visual>
-      <collision>
-        <origin xyz="9.06e-05 -0.0010859 -0.0010079" rpy="0. 0.8801533 -3.141593" />
-        <geometry>
-          <mesh filename="package://igvc_test_description/meshes/left_wheel_link__in_Wheel_Stand_In_01__in_Wheel_Stand_In.obj" scale="1. 1. 1." />
-        </geometry>
-      </collision>
+      <!-- SIM: cylinder, not the mesh. Two independent reasons.
+           1. The mesh CRASHES the physics engine. Verified 2026-09-15:
+              left_wheel, right_wheel, caster_wheel and caster_raceway have
+              528, 528, 500 and 209 vertices and ZERO vertex normals. dartsim
+              reports "does not have a normal count [0] that matches its
+              vertex count [3168]. This submesh will be ignored!", then
+              segfaults in OdeMesh::fillArrays on the empty result. gz sim
+              dies on the first physics step, exit 139. Those four are exactly
+              the parts that must collide for the robot to move.
+           2. Even repaired, a faceted mesh is a poor wheel: it rolls on flats
+              and catches on edges. RQ-11 makes the same point about cost.
+           Radius 0.1016 and width 0.0640 are the mesh's own measured bounding
+           box (0.2032 x 0.0640 x 0.2032), so 0.2032 is the DIAMETER. See the
+           long note in urdf/gazebo/gazebo_sim.urdf.xacro. The rpy rotates the
+           cylinder's Z axis onto Y, which is the wheel joint axis.
+           The real robot keeps the mesh, below. -->
+      <xacro:if value="$(arg sim)">
+        <collision>
+          <origin xyz="0. 0. 0." rpy="1.5707963 0. 0." />
+          <geometry>
+            <cylinder radius="0.1016" length="0.0640" />
+          </geometry>
+        </collision>
+      </xacro:if>
+      <xacro:unless value="$(arg sim)">
+        <collision>
+          <origin xyz="9.06e-05 -0.0010859 -0.0010079" rpy="0. 0.8801533 -3.141593" />
+          <geometry>
+            <mesh filename="package://igvc_test_description/meshes/left_wheel_link__in_Wheel_Stand_In_01__in_Wheel_Stand_In.obj" scale="1. 1. 1." />
+          </geometry>
+        </collision>
+      </xacro:unless>
     </link>
     <link name="right_wheel_link">
@@ -101,10 +150,21 @@
         </geometry>
       </visual>
-      <collision>
-        <origin xyz="-0.0007409 0.0085441 0.0012195" rpy="-3.141593 0. -7.32051e-08" />
-        <geometry>
-          <mesh filename="package://igvc_test_description/meshes/right_wheel_link__in_Wheel_Stand_In_01__in_Wheel_Stand_In.obj" scale="1. 1. 1." />
-        </geometry>
-      </collision>
+      <!-- SIM: cylinder. Same reasoning as left_wheel_link above. -->
+      <xacro:if value="$(arg sim)">
+        <collision>
+          <origin xyz="0. 0. 0." rpy="1.5707963 0. 0." />
+          <geometry>
+            <cylinder radius="0.1016" length="0.0640" />
+          </geometry>
+        </collision>
+      </xacro:if>
+      <xacro:unless value="$(arg sim)">
+        <collision>
+          <origin xyz="-0.0007409 0.0085441 0.0012195" rpy="-3.141593 0. -7.32051e-08" />
+          <geometry>
+            <mesh filename="package://igvc_test_description/meshes/right_wheel_link__in_Wheel_Stand_In_01__in_Wheel_Stand_In.obj" scale="1. 1. 1." />
+          </geometry>
+        </collision>
+      </xacro:unless>
     </link>
     <link name="chassis_link">

File: src/igvc_test_description/urdf/robots/test_robot.urdf.xacro (robot description, xacro)
@@ -1,4 +1,10 @@
 <?xml version="1.0" encoding="UTF-8"?>
 <robot xmlns:xacro="http://www.ros.org/wiki/xacro" name='igvc_test_robot'>
+    <!-- Declared FIRST, before any include or macro call, because
+         test_robot_body.urdf.xacro reads $(arg sim) to choose primitive
+         collision shapes over the mesh ones. xacro evaluates $(arg) at macro
+         invocation time, and <xacro:robot_body /> below runs before the
+         declaration that used to sit at the bottom of this file. -->
+    <xacro:arg name="sim" default="false" />
     <xacro:include filename="$(find igvc_test_description)/urdf/parts/test_robot_body.urdf.xacro" />
     <xacro:include filename="$(find igvc_test_description)/urdf/control/ros2_control_info.urdf.xacro" />
@@ -24,6 +30,6 @@
     </xacro:gps_antenna>
     <!-- Gazebo-only plugins and sensors. Inert on the real robot: pass
-         sim:=true to load them. See urdf/gazebo/gazebo_sim.urdf.xacro. -->
-    <xacro:arg name="sim" default="false" />
+         sim:=true to load them. See urdf/gazebo/gazebo_sim.urdf.xacro.
+         The sim arg itself is declared at the top of this file. -->
     <xacro:if value="$(arg sim)">
         <xacro:include filename="$(find igvc_test_description)/urdf/gazebo/gazebo_sim.urdf.xacro" />
