Commit message: Reject an unrecognised sim_cameras instead of building a robot with none
The camera dispatch in gazebo_sim.urdf.xacro was two xacro:if blocks comparing
a string to literals, with no else branch. Any value that was not none, front or
all produced a robot with zero cameras that converted to valid SDF, spawned
cleanly, passed every topic-name check in the smoke test, and failed only much
later as "the lane detector sees nothing". sim_cameras:=fron was a silent wrong
answer.

Two guards, because there are two ways in. gazebo_sim.launch.py raises a
readable RuntimeError before xacro is invoked, which is the path everyone
actually uses. gazebo_sim.urdf.xacro validates with list.index(), which raises a
ValueError naming the offending value, for anyone running xacro by hand.

The xacro guard had to be made load-bearing to work at all. A validation
property that nothing reads is never evaluated, because xacro evaluates
properties lazily, so the first version of this passed every bad value through
untouched. The dispatch now switches on the validated index itself
(cams_idx >= 1, cams_idx == 2), so it cannot be skipped.

Verified, with the workspace built and sourced, against the installed xacro:

  front        exit 0, 1 rgbd camera
  all          exit 0, 3 rgbd cameras
  none         exit 0, 0 rgbd cameras
  fron         exit 2, rejected
  front,left   exit 2, rejected
  true         exit 2, rejected

An earlier run of that same test reported all six as rejected, including the
three valid ones, because the workspace was not sourced and the package was not
in the ament index. It looked like a pass. Checking the error text rather than
the exit code is what caught it.

Co-Authored-By: Claude Opus 5 <noreply@anthropic.com>

File: src/igvc_test_description/urdf/gazebo/gazebo_sim.urdf.xacro (robot description, xacro)
@@ -24,4 +24,19 @@
   <xacro:arg name="sim_camera_hz"     default="15" />
   <xacro:property name="cams" value="$(arg sim_cameras)" />
+  <!-- Reject an unrecognised sim_cameras here, not silently.
+       The camera dispatch below used to be two xacro:if blocks comparing cams
+       to string literals, with no else, so a typo like "fron" or "front,left"
+       produced a robot with NO cameras that converted to valid SDF and spawned
+       without a single warning.
+       list.index() raises a ValueError naming the offending value, which is
+       the loudest thing xacro offers. It has to be USED to fire: xacro
+       evaluates properties lazily, so a validation property nothing reads is
+       never evaluated (found the hard way, 2026-09-17). cams_idx is therefore
+       what the dispatch itself switches on: none=0, front=1, all=2.
+       gazebo_sim.launch.py checks the same set and raises a friendlier message
+       before xacro is ever invoked; this guard is for anyone running xacro by
+       hand. -->
+  <xacro:property name="cams_idx"
+                  value="${['none','front','all'].index(cams)}" />
   <!-- Geometry measured from the model, not copied from controllers.yaml.
        Both values there are wrong for simulation, and one of them looks wrong
@@ -185,8 +200,8 @@
     </gazebo>
   </xacro:macro>
-  <xacro:if value="${cams == 'front' or cams == 'all'}">
+  <xacro:if value="${cams_idx >= 1}">   <!-- front or all -->
     <xacro:sim_rgbd prefix="front" />
   </xacro:if>
-  <xacro:if value="${cams == 'all'}">
+  <xacro:if value="${cams_idx == 2}">   <!-- all -->
     <xacro:sim_rgbd prefix="left" />
     <xacro:sim_rgbd prefix="right" />

Commit message: Simulator: DiffDrive wheel geometry as xacro arguments, 2026 values the default
gazebo_sim.urdf.xacro hard-coded the 2026 robot's wheel separation (0.57633)
and radius (0.1016). They are now the defaults of sim_wheel_separation and
sim_wheel_radius, so a robot description that declares those arguments first
(xacro keeps the first default it sees) can pass its own measured geometry.

The 2026 robot is unchanged: its expanded description (sim, real, and
sim_cameras:=all) is byte-identical to before, 0 differing lines apart from
the "autogenerated" comment.

Co-Authored-By: Claude Opus 5.5 <noreply@anthropic.com>

File: src/igvc_test_description/urdf/gazebo/gazebo_sim.urdf.xacro (robot description, xacro)
@@ -52,7 +52,13 @@
        floating 97 mm in the air.
        separation 0.57633 = 0.2844359 + 0.2918941 from the wheel joint origins.
-       controllers.yaml says 0.5027, which is 0.87x the geometry it describes. -->
-  <xacro:property name="wheel_separation" value="0.57633" />
-  <xacro:property name="wheel_radius"     value="0.1016" />
+       controllers.yaml says 0.5027, which is 0.87x the geometry it describes.
+       Arguments, so the 2027 robot (urdf/robot_2027/igvc_2027.urdf.xacro) can
+       pass its own measured geometry. It declares them first, and xacro keeps
+       the first default it sees, so the 2026 robot gets exactly the values
+       above. -->
+  <xacro:arg name="sim_wheel_separation" default="0.57633" />
+  <xacro:arg name="sim_wheel_radius"     default="0.1016" />
+  <xacro:property name="wheel_separation" value="$(arg sim_wheel_separation)" />
+  <xacro:property name="wheel_radius"     value="$(arg sim_wheel_radius)" />
 <!-- ================= drive =================
        Both wheel joints have axis 0 1 0, so both take a positive radius here.
